Commit message: Changes description package to odri_bolt_description.

File: odri_bolt_description/ros2_control/system_bolt.ros2_control.xacro (robot description, xacro)
@@ -20,5 +20,5 @@
             <plugin>ros2_control_odri/SystemOdriHardware</plugin>
             <param name="bolt_yaml">2.0</param>
-            <xacro:property name="prop_bolt_config_yaml" value="$(find ros2_description_bolt)/config/bolt_config.yaml" />
+            <xacro:property name="prop_bolt_config_yaml" value="$(find odri_bolt_description)/config/bolt_config.yaml" />
             <param name="odri_config_yaml">${prop_bolt_config_yaml}</param>
             <param name="desired_starting_position">0.0 0.0 0.0 0.0 0.0 0.0</param>

File: odri_bolt_description/urdf/leg.xacro (robot description, xacro)
@@ -78,8 +78,8 @@
                 <geometry>
                     <xacro:unless value="${is_right}">
-                        <mesh filename="file://$(find ros2_description_bolt)/meshes/${mesh_ext}/bolt_hip_fe_left_side.${mesh_ext}"/>
+                        <mesh filename="file://$(find odri_bolt_description)/meshes/${mesh_ext}/bolt_hip_fe_left_side.${mesh_ext}"/>
                     </xacro:unless>
                     <xacro:if value="${is_right}">
-                        <mesh filename="file://$(find ros2_description_bolt)/meshes/${mesh_ext}/bolt_hip_fe_right_side.${mesh_ext}"/>
+                        <mesh filename="file://$(find odri_bolt_description)/meshes/${mesh_ext}/bolt_hip_fe_right_side.${mesh_ext}"/>
                     </xacro:if>
                 </geometry>
@@ -93,8 +93,8 @@
                 <geometry>
                     <xacro:unless value="${is_right}">
-                        <mesh filename="file://$(find ros2_description_bolt)/meshes/${mesh_ext}/bolt_hip_fe_left_side.${mesh_ext}"/>
+                        <mesh filename="file://$(find odri_bolt_description)/meshes/${mesh_ext}/bolt_hip_fe_left_side.${mesh_ext}"/>
                     </xacro:unless>
                     <xacro:if value="${is_right}">
-                        <mesh filename="file://$(find ros2_description_bolt)/meshes/${mesh_ext}/bolt_hip_fe_right_side.${mesh_ext}"/>
+                        <mesh filename="file://$(find odri_bolt_description)/meshes/${mesh_ext}/bolt_hip_fe_right_side.${mesh_ext}"/>
                     </xacro:if>
                 </geometry>
@@ -159,16 +159,16 @@
                     <xacro:unless value="${new_leg}">
                         <xacro:unless value="${is_right}">
-                            <mesh filename="file://$(find ros2_description_bolt)/meshes/${mesh_ext}/bolt_upper_leg_left_side.${mesh_ext}"/>
-                        </xacro:unless>
-                        <xacro:if value="${is_right}">
-                            <mesh filename="file://$(find ros2_description_bolt)/meshes/${mesh_ext}/bolt_upper_leg_right_side.${mesh_ext}"/>
+                            <mesh filename="file://$(find odri_bolt_description)/meshes/${mesh_ext}/bolt_upper_leg_left_side.${mesh_ext}"/>
+                        </xacro:unless>
+                        <xacro:if value="${is_right}">
+                            <mesh filename="file://$(find odri_bolt_description)/meshes/${mesh_ext}/bolt_upper_leg_right_side.${mesh_ext}"/>
                         </xacro:if>
                     </xacro:unless>
                     <xacro:if value="${new_leg}">
                         <xacro:unless value="${is_right}">
-                            <mesh filename="file://$(find ros2_description_bolt)/meshes/${mesh_ext}/upper_leg_200mm_left_side.${mesh_ext}"/>
-                        </xacro:unless>
-                        <xacro:if value="${is_right}">
-                            <mesh filename="file://$(find ros2_description_bolt)/meshes/${mesh_ext}/upper_leg_200mm_right_side.${mesh_ext}"/>
+                            <mesh filename="file://$(find odri_bolt_description)/meshes/${mesh_ext}/upper_leg_200mm_left_side.${mesh_ext}"/>
+                        </xacro:unless>
+                        <xacro:if value="${is_right}">
+                            <mesh filename="file://$(find odri_bolt_description)/meshes/${mesh_ext}/upper_leg_200mm_right_side.${mesh_ext}"/>
                         </xacro:if>
                     </xacro:if>
@@ -184,16 +184,16 @@
                     <xacro:unless value="${new_leg}">
                         <xacro:unless value="${is_right}">
-                            <mesh filename="file://$(find ros2_description_bolt)/meshes/${mesh_ext}/bolt_upper_leg_left_side.${mesh_ext}"/>
-                        </xacro:unless>
-                        <xacro:if value="${is_right}">
-                            <mesh filename="file://$(find ros2_description_bolt)/meshes/${mesh_ext}/bolt_upper_leg_right_side.${mesh_ext}"/>
+                            <mesh filename="file://$(find odri_bolt_description)/meshes/${mesh_ext}/bolt_upper_leg_left_side.${mesh_ext}"/>
+                        </xacro:unless>
+                        <xacro:if value="${is_right}">
+                            <mesh filename="file://$(find odri_bolt_description)/meshes/${mesh_ext}/bolt_upper_leg_right_side.${mesh_ext}"/>
                         </xacro:if>
                     </xacro:unless>
                     <xacro:if value="${new_leg}">
                         <xacro:unless value="${is_right}">
-                            <mesh filename="file://$(find ros2_description_bolt)/meshes/${mesh_ext}/upper_leg_200mm_left_side.${mesh_ext}"/>
-                        </xacro:unless>
-                        <xacro:if value="${is_right}">
-                            <mesh filename="file://$(find ros2_description_bolt)/meshes/${mesh_ext}/upper_leg_200mm_right_side.${mesh_ext}"/>
+                            <mesh filename="file://$(find odri_bolt_description)/meshes/${mesh_ext}/upper_leg_200mm_left_side.${mesh_ext}"/>
+                        </xacro:unless>
+                        <xacro:if value="${is_right}">
+                            <mesh filename="file://$(find odri_bolt_description)/meshes/${mesh_ext}/upper_leg_200mm_right_side.${mesh_ext}"/>
                         </xacro:if>
                     </xacro:if>
@@ -261,16 +261,16 @@
                     <xacro:unless value="${new_leg}">
                         <xacro:unless value="${is_right}">
-                            <mesh filename="file://$(find ros2_description_bolt)/meshes/${mesh_ext}/bolt_lower_leg_left_side.${mesh_ext}"/>
-                        </xacro:unless>
-                        <xacro:if value="${is_right}">
-                            <mesh filename="file://$(find ros2_description_bolt)/meshes/${mesh_ext}/bolt_lower_leg_right_side.${mesh_ext}"/>
+                            <mesh filename="file://$(find odri_bolt_description)/meshes/${mesh_ext}/bolt_lower_leg_left_side.${mesh_ext}"/>
+                        </xacro:unless>
+                        <xacro:if value="${is_right}">
+                            <mesh filename="file://$(find odri_bolt_description)/meshes/${mesh_ext}/bolt_lower_leg_right_side.${mesh_ext}"/>
                         </xacro:if>
                     </xacro:unless>
                     <xacro:if value="${new_leg}">
                         <xacro:unless value="${is_right}">
-                            <mesh filename="file://$(find ros2_description_bolt)/meshes/${mesh_ext}/lower_leg_200mm_left_side.${mesh_ext}"/>
-                        </xacro:unless>
-                        <xacro:if value="${is_right}">
-                            <mesh filename="file://$(find ros2_description_bolt)/meshes/${mesh_ext}/lower_leg_200mm_right_side.${mesh_ext}"/>
+                            <mesh filename="file://$(find odri_bolt_description)/meshes/${mesh_ext}/lower_leg_200mm_left_side.${mesh_ext}"/>
+                        </xacro:unless>
+                        <xacro:if value="${is_right}">
+                            <mesh filename="file://$(find odri_bolt_description)/meshes/${mesh_ext}/lower_leg_200mm_right_side.${mesh_ext}"/>
                         </xacro:if>
                     </xacro:if>
@@ -286,16 +286,16 @@
                     <xacro:unless value="${new_leg}">
                         <xacro:unless value="${is_right}">
-                            <mesh filename="file://$(find ros2_description_bolt)/meshes/${mesh_ext}/bolt_lower_leg_left_side.${mesh_ext}"/>
-                        </xacro:unless>
-                        <xacro:if value="${is_right}">
-                            <mesh filename="file://$(find ros2_description_bolt)/meshes/${mesh_ext}/bolt_lower_leg_right_side.${mesh_ext}"/>
+                            <mesh filename="file://$(find odri_bolt_description)/meshes/${mesh_ext}/bolt_lower_leg_left_side.${mesh_ext}"/>
+                        </xacro:unless>
+                        <xacro:if value="${is_right}">
+                            <mesh filename="file://$(find odri_bolt_description)/meshes/${mesh_ext}/bolt_lower_leg_right_side.${mesh_ext}"/>
                         </xacro:if>
                     </xacro:unless>
                     <xacro:if value="${new_leg}">
                         <xacro:unless value="${is_right}">
-                            <mesh filename="file://$(find ros2_description_bolt)/meshes/${mesh_ext}/lower_leg_200mm_left_side.${mesh_ext}"/>
-                        </xacro:unless>
-                        <xacro:if value="${is_right}">
-                            <mesh filename="file://$(find ros2_description_bolt)/meshes/${mesh_ext}/lower_leg_200mm_right_side.${mesh_ext}"/>
+                            <mesh filename="file://$(find odri_bolt_description)/meshes/${mesh_ext}/lower_leg_200mm_left_side.${mesh_ext}"/>
+                        </xacro:unless>
+                        <xacro:if value="${is_right}">
+                            <mesh filename="file://$(find odri_bolt_description)/meshes/${mesh_ext}/lower_leg_200mm_right_side.${mesh_ext}"/>
                         </xacro:if>
                     </xacro:if>
@@ -363,5 +363,5 @@
                     </xacro:if>
                     <xacro:unless value="${has_passive_ankle}">
-                        <mesh filename="file://$(find ros2_description_bolt)/meshes/${mesh_ext}/bolt_foot.${mesh_ext}"/>
+                        <mesh filename="file://$(find odri_bolt_description)/meshes/${mesh_ext}/bolt_foot.${mesh_ext}"/>
                     </xacro:unless>
                 </geometry>
@@ -383,5 +383,5 @@
                     </xacro:if>
                     <xacro:unless value="${has_passive_ankle}">
-                        <mesh filename="file://$(find ros2_description_bolt)/meshes/${mesh_ext}/bolt_foot.${mesh_ext}"/>
+                        <mesh filename="file://$(find odri_bolt_description)/meshes/${mesh_ext}/bolt_foot.${mesh_ext}"/>
                     </xacro:unless>
                 </geometry>

File: odri_bolt_description/urdf/system_bolt.urdf.xacro (robot description, xacro)
@@ -26,5 +26,5 @@
           <origin xyz="0 0 0" rpy="0 0 0" />
           <geometry>
-            <mesh filename="file://$(find ros2_description_bolt)/meshes/${mesh_ext}/bolt_body.${mesh_ext}"/>
+            <mesh filename="file://$(find odri_bolt_description)/meshes/${mesh_ext}/bolt_body.${mesh_ext}"/>
           </geometry>
           <material name="${color_name}">
@@ -36,5 +36,5 @@
           <origin xyz="0 0 0" rpy="0 0 0" />
           <geometry>
-            <mesh filename="file://$(find ros2_description_bolt)/meshes/${mesh_ext}/bolt_body.${mesh_ext}"/>
+            <mesh filename="file://$(find odri_bolt_description)/meshes/${mesh_ext}/bolt_body.${mesh_ext}"/>
           </geometry>
           <material name="${color_name}">

File: odri_bolt_description/urdf/system_bolt_description.urdf.xacro (robot description, xacro)
@@ -24,8 +24,8 @@
   <xacro:if value="$(arg use_sim)">
     <xacro:if value="$(arg use_crane)">
-      <xacro:include filename="$(find ros2_description_bolt)/urdf/crane.urdf.xacro" />
+      <xacro:include filename="$(find odri_bolt_description)/urdf/crane.urdf.xacro" />
     </xacro:if>
   </xacro:if>
-  <xacro:include filename="$(find ros2_description_bolt)/ros2_control/system_bolt.ros2_control.xacro" />
+  <xacro:include filename="$(find odri_bolt_description)/ros2_control/system_bolt.ros2_control.xacro" />
   <!-- ros_control plugin for Gazebo -->
   <xacro:if value="$(arg use_sim)">
