Commit message: Update to depend to gz_ros2_control_bolt Mistake this should be gz_ros2_control_odri. Keep it just for bookmarking.

File: odri_bolt_description/gazebo/bolt.gazebo.xacro (robot description, xacro)
@@ -11,5 +11,5 @@
     <gazebo>
       <plugin name="gz_ros2_control::GazeboSimROS2ControlPlugin" filename="gz_ros2_control-system">
-	<parameters>$(find gazebo_ros2_control_bolt)/config/bolt_gazebo_config_controller.yaml</parameters>
+	<parameters>$(find odri_bolt_gz)/config/odri_bolt_controllers.yaml</parameters>
         <controller_manager_node_name>${prefix}controller_manager</controller_manager_node_name>
       </plugin>

File: odri_bolt_description/ros2_control/system_bolt.ros2_control.xacro (robot description, xacro)
@@ -1,14 +1,14 @@
 <?xml version="1.0"?>
 <robot xmlns:xacro="http://www.ros.org/wiki/xacro">
-  <xacro:macro name="system_bolt_ros2_control" params="name prefix use_sim:=^|false use_fake_hardware:=^|true fake_sensor_commands:=^|false slowdown:=2.0 ethernet_port:=^|enp6s0f1 true:=^|true false:=^|false">
+  <xacro:macro name="system_bolt_ros2_control" params="name prefix use_gazebo_sim:=^|false use_fake_hardware:=^|true fake_sensor_commands:=^|false slowdown:=2.0 ethernet_port:=^|enp6s0f1 true:=^|true false:=^|false">
     <ros2_control name="${name}" type="system">
-      <xacro:if value="$(arg use_sim)">
+      <xacro:if value="$(arg use_gazebo_sim)">
         <hardware>
-          <plugin>gazebo_ros2_control_bolt/GazeboBoltSystem</plugin>
+          <plugin>gz_ros2_control/GazeboBoltSimSystem</plugin>
 	  <param name="default_kp">1000.0</param>
 	  <param name="default_kd">10.0</param>
         </hardware>
       </xacro:if>
-      <xacro:unless value="$(arg use_sim)">
+      <xacro:unless value="$(arg use_gazebo_sim)">
         <hardware>
           <xacro:if value="${use_fake_hardware}">

File: odri_bolt_description/urdf/system_bolt_description.urdf.xacro (robot description, xacro)
@@ -44,10 +44,8 @@
   <xacro:system_bolt_ros2_control
     name="SystemBoltRos2Control" prefix="$(arg prefix)" use_fake_hardware="$(arg use_fake_hardware)"
-      use_sim="$(arg use_sim)"/>
-    <!-- ros_control plugin for Gazebo -->
-    <xacro:if value="$(arg use_gazebo_sim)">
-      <xacro:odri_bolt_gazebo
-          name="OdriBoltGazeboRos2Control" prefix="$(arg prefix)"
-          />
+      use_gazebo_sim="$(arg use_gazebo_sim)"/>
+  <!-- ros_control plugin for Gazebo -->
+  <xacro:if value="$(arg use_gazebo_sim)">
+    <xacro:odri_bolt_gazebo prefix="$(arg prefix)" />
   </xacro:if>
 </robot>

Commit message: [odri_bolt_description] Update name of the odri namespace [odri_bolt_gz] Simulation

File: odri_bolt_description/gazebo/bolt.gazebo.xacro (robot description, xacro)
@@ -10,5 +10,5 @@
     </gazebo>
     <gazebo>
-      <plugin name="gz_ros2_control::GazeboSimROS2ControlPlugin" filename="gz_ros2_control-system">
+      <plugin name="odri_gz_ros2_control::GazeboOdriSimROS2ControlPlugin" filename="odri_gz_ros2_control-system">
 	<parameters>$(find odri_bolt_gz)/config/odri_bolt_controllers.yaml</parameters>
         <controller_manager_node_name>${prefix}controller_manager</controller_manager_node_name>

File: odri_bolt_description/ros2_control/system_bolt.ros2_control.xacro (robot description, xacro)
@@ -5,5 +5,5 @@
       <xacro:if value="$(arg use_gazebo_sim)">
         <hardware>
-          <plugin>gz_ros2_control/GazeboOdriSimSystem</plugin>
+          <plugin>odri_gz_ros2_control/GazeboOdriSimSystem</plugin>
 	  <param name="default_kp">1000.0</param>
 	  <param name="default_kd">10.0</param>

File: odri_bolt_description/urdf/crane.urdf.xacro (robot description, xacro)
@@ -41,5 +41,5 @@
     <link name="world"/>
     <joint name="fixed" type="fixed">
-      <origin xyz="0.0 0.0 0.2" rpy="0.0  0.0  0.0"/>
+      <origin xyz="0.0 0.0 0.6" rpy="0.0  0.0  0.0"/>
       <parent link="world"/>
       <child link="crane_link"/>
